Commit message: code refactoring

File: src/multi_jackal/multi_jackal_description/urdf/jackal.urdf.xacro (robot description, xacro)
@@ -60,5 +60,5 @@
       <type>transmission_interface/SimpleTransmission</type>
       <joint name="${prefix}_wheel">
-        <hardwareInterface>VelocityJointInterface</hardwareInterface>
+        <hardwareInterface>hardware_interface/VelocityJointInterface</hardwareInterface>
       </joint>
       <actuator name="${prefix}_actuator">
@@ -121,4 +121,5 @@
   </link>
   <joint name="fenders_joint" type="fixed">
+    <!-- <origin xyz="0 0 0" rpy="0 0 0"/>  -->
     <parent link="chassis_link" />
     <child link="fenders_link" />
@@ -174,7 +175,7 @@
   <!-- Bring in simulation data for Gazebo. -->
   <xacro:include filename="jackal.gazebo" />
-  <!-- Optional standard accessories, as supplied by Clearpath.-->
+  <!-- Optional standard accessories, as supplied by Clearpath. 加载激光雷达和相机-->
   <xacro:include filename="base_accessories.urdf.xacro" />
-  <!-- Optional custom accessories. -->
+  <!-- Optional custom accessories. 加载动态障碍物的模型-->
   <xacro:include filename="custom_accessories.urdf.xacro" />
 </robot>
